File: kicad/demeter.sch (KiCad schematic (older format))
At the start: 13 parts, among them IC1 ATMEGA328-P, K1 DHT22, P1 POWER, P2 RELAYS, P3 SD_RTC, P4 LDR, P5 RS232, SW1 PUSH

Commit message: Esquemáticos Kicad
Parts:
- removed P5: RS232, symbol CONN_4
- added K1: SW_IPS, symbol CONN_3
- added P5: RS232, symbol CONN_6
- renumbered K1 to K2, P3 to P2, P2 to P3, R3 to R2, R2 to R3
Connections:
- net GND: now also P2.10, P2.8, P5.6; no longer P2.1, P2.3
- net MISO-SD: now also P2.9; no longer P2.7
- net MOSI-SD: now also P2.1; no longer P2.9
- net RX-BT: now also P5.2
- net SCK-SD: now also P2.7; no longer P2.5
- net SCL-RTC: now also P2.4; no longer P2.2
- net SDA-RTC: now also P2.6; no longer P2.4
- net SS-SD: now also P2.3; no longer P2.6
- net TX-BT: now also P5.3
- net VCC: now also P2.2, K1.3 (P3), P5.4; no longer P2.10, P2.8
- net RST: now reaches IC1.1 ((PCINT14/~RESET~)PC6)
- net RST: now also K1.1 (P1)
- new net: K1.2 (PM), P2.5
- no-connect marks 10 -> 11
Other:
- moved on the sheet: K2, P2, R3
